File: Armageddon/Armageddon.kicad_sch (KiCad schematic)
At the start: 33 parts, among them J1 XT60PW-M, J2 530470610, U2 PTPS16850VMAR

Commit message: Added +5V Rail
Parts:
- added C14, C20: 10uF, Capacitor_SMD:C_0805_2012Metric_Pad1.18x1.45mm_HandSolder, symbol Device:C
- added C15, C21: 100nF, Capacitor_SMD:C_0603_1608Metric_Pad1.08x0.95mm_HandSolder, symbol Device:C
- added C16: 22pF, Capacitor_SMD:C_0603_1608Metric_Pad1.08x0.95mm_HandSolder, symbol Device:C
- added C17, C18, C19: 47uF, Capacitor_SMD:C_0805_2012Metric_Pad1.18x1.45mm_HandSolder, symbol Device:C
- added R13: 187K, Resistor_SMD:R_0603_1608Metric_Pad0.98x0.95mm_HandSolder, symbol Device:R
- added R14: 49.9K, Resistor_SMD:R_0603_1608Metric_Pad0.98x0.95mm_HandSolder, symbol Device:R
- added R15, R18: 100K, Resistor_SMD:R_0603_1608Metric_Pad0.98x0.95mm_HandSolder, symbol Device:R
- added R16: 15.8K, Resistor_SMD:R_0603_1608Metric_Pad0.98x0.95mm_HandSolder, symbol Device:R
- added R17: 24.9K, Resistor_SMD:R_0603_1608Metric_Pad0.98x0.95mm_HandSolder, symbol Device:R
- added U1: TLVM13610RDFR, RDF0022A-MFG, symbol TVLM13610:TLVM13610RDFR
Connections:
- net +24V: now also C14.1, C15.1, R13.1, U1.1 (VIN)
- net GND: now also C14.2, C15.2, C17.2, C18.2, C19.2, C20.2, C21.2, R14.2, R16.2, R17.2, U1.11 (AGND), U1.14 (AGND), U1.15 (AGND), U1.19 (PGND), U1.20 (PGND), U1.21 (AGND), U1.22 (AGND), U1.7 (AGND)
- new net: R16.1, U1.12 (RT)
- new net: R13.2, R14.1, U1.17 (EN)
- new net: C20.1, C21.1, U1.18 (VIN)
- new net: U1.2 (RBOOT), U1.3 (CBOOT)
- new net: R15.2, U1.6 (VCC)
- new net: C16.2, R17.1, R18.2, U1.8 (FB)
- new net +5V: C16.1, C17.1, C18.1, C19.1, R18.1, U1.10 (VOUT), U1.5 (VLDOIN), U1.9 (VOUT)
- new net 5VGOOD: R15.1, U1.13 (PG)
Other:
- note added: "5V Rail 8A"
- moved on the sheet: C1, C10, C11, C12, C13, C2, C3, C4, C5, C6, C7, C8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
