File: Armageddon/Armageddon.kicad_sch (KiCad schematic)
At the start: 48 parts, among them J1 XT60PW-M, J2 530470610, U1 TLVM13610RDFR, U2 PTPS16850VMAR

Commit message: EFUSE REMOVED
Parts:
- removed C10, C4, C5, C8: 100pF, Capacitor_SMD:C_0603_1608Metric_Pad1.08x0.95mm_HandSolder, symbol Device:C
- removed C11, C13: 22pF, Capacitor_SMD:C_0603_1608Metric_Pad1.08x0.95mm_HandSolder, symbol Device:C
- removed C12: 4.7nF/50V, Capacitor_SMD:C_0603_1608Metric_Pad1.08x0.95mm_HandSolder, symbol Device:C
- removed C3: 220nF/50V, Capacitor_SMD:C_0805_2012Metric, symbol Device:C_Small
- removed C6: 100nF/50V, Capacitor_SMD:C_0805_2012Metric, symbol Device:C_Small
- removed C7: 22uF/50V, Capacitor_SMD:C_2220_5750Metric_Pad1.97x5.40mm_HandSolder, symbol Device:C
- removed C9: 47nF/50V, Capacitor_SMD:C_0603_1608Metric_Pad1.08x0.95mm_HandSolder, symbol Device:C
- removed CR1: MMSZ5231B-7-F, SOD123_DIO, symbol MMSZ5231B_7_F:MMSZ5231B-7-F
- removed D2: SMAJ28A, Diode_SMD:D_SMA, symbol Diode:SMAJ28A
- removed R1: 150R, Resistor_SMD:R_0805_2012Metric, symbol Device:R
- removed R10: 40.2K/0.1%, Resistor_SMD:R_0603_1608Metric_Pad0.98x0.95mm_HandSolder, symbol Device:R
- removed R11: 3.92K/0.1%, Resistor_SMD:R_0603_1608Metric_Pad0.98x0.95mm_HandSolder, symbol Device:R
- removed R12: 1.5K, Resistor_SMD:R_0603_1608Metric_Pad0.98x0.95mm_HandSolder, symbol Device:R
- removed R2: 750K, Resistor_SMD:R_0603_1608Metric_Pad0.98x0.95mm_HandSolder, symbol Device:R
- removed R3: 100K, Resistor_SMD:R_0603_1608Metric_Pad0.98x0.95mm_HandSolder, symbol Device:R
- removed R4: 330K, Resistor_SMD:R_0603_1608Metric_Pad0.98x0.95mm_HandSolder, symbol Device:R
- removed R5: 720K, Resistor_SMD:R_0603_1608Metric_Pad0.98x0.95mm_HandSolder, symbol Device:R
- removed R6: 30K, Resistor_SMD:R_0603_1608Metric_Pad0.98x0.95mm_HandSolder, symbol Device:R
- removed R7, R8: 1K, Resistor_SMD:R_0603_1608Metric_Pad0.98x0.95mm_HandSolder, symbol Device:R
- removed R9: 3K9, Resistor_SMD:R_0603_1608Metric_Pad0.98x0.95mm_HandSolder, symbol Device:R
- removed TP1, TP2: TestPoint_Alt, symbol Connector:TestPoint_Alt
- removed U2: PTPS16850VMAR, VMA0023A-MFG, symbol TPS16850VMAR:PTPS16850VMAR
Connections:
- net 24V Vin is gone; now on net +24V: C1.1, C2.1, D1.1 (A1), J1.1 (P)
- net GND: no longer J2.6
- net PFault: no longer names the net of J2.4
- net PWR PB+: no longer names the net of J2.1
- net PWR PB-: no longer names the net of J2.2
- net Pgood: no longer names the net of J2.5
- net R_LED_A: no longer names the net of J2.3
Other:
- note added: "24V in"
- note removed: "24V in + EFuse"
- note removed: "IOCP: 15A"
- note removed: "Iocp * 1.5"
- note removed: "OVPR: 30V"
- note removed: "To G LED A"
- note removed: "To G LED K"
- note removed: "To R LED K"
- note removed: "UVLO 10V"
- moved on the sheet: C1, C14, C15, C16, C17, C18, C19, C20, C21, D1, J1, J2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
