File: Armageddon/RP Compute Module.kicad_sch (KiCad schematic)
At the start: 1 part, among them U3 CM5108032

Commit message: Updated Molex USB C Symbol
Parts:
- removed U3: CM5108032, CM5108032:MODULE_CM5108032, symbol CM5108032:CM5108032
