File: LogicAnalyzer_RP2350/LogicAnalyzer_RP2350/LevelShifters.kicad_sch (KiCad schematic)
At the start: 0 parts

Commit message: Added Level Shifter TXU Series
Parts:
- added U10, U5, U6, U7, U8, U9: TXU0104PWR, TSSOP_0104PWR_TEX, symbol TXU0104PWR:TXU0104PWR
Connections:
- new net D1: U5.2 (A1)
- new net D10: U7.3 (A2)
- new net D11: U7.4 (A3)
- new net D12: U7.5 (A4)
- new net D13: U8.2 (A1)
- new net D14: U8.3 (A2)
- new net D15: U8.4 (A3)
- new net D16: U8.5 (A4)
- new net D17: U9.2 (A1)
- new net D18: U9.3 (A2)
- new net D19: U9.4 (A3)
- new net D2: U5.3 (A2)
- new net D20: U9.5 (A4)
- new net D21: U10.2 (A1)
- new net D22: U10.3 (A2)
- new net D23: U10.4 (A3)
- new net D24: U10.5 (A4)
- new net D3: U5.4 (A3)
- new net D4: U5.5 (A4)
- new net D5: U6.2 (A1)
- new net D6: U6.3 (A2)
- new net D7: U6.4 (A3)
- new net D8: U6.5 (A4)
- new net D9: U7.2 (A1)

Commit message: Added Level Shifter Connections
Parts:
- added C27, C28, C29, C30, C31, C32, C33, C34, C35, C36, C37, C38, C39, C40, C41, C42, C43: 100nF, Capacitor_SMD:C_0603_1608Metric_Pad1.08x0.95mm_HandSolder, symbol Device:C_Small
- added J4: IPL1-115-01-X-D-RA-K, IPL1-115-01-X-D-RA-K:SAMTEC_IPL1-115-01-X-D-RA-K, symbol IPL1-115-01-X-D-RA-K:IPL1-115-01-X-D-RA-K
Connections:
- net VREF: now reaches U7.1 (VCCA)
- net VREF: now also U10.1 (VCCA), U5.1 (VCCA), U6.1 (VCCA), U8.1 (VCCA), U9.1 (VCCA), C27.1, C28.1, C29.1, C30.1, C31.1, C32.1
- net DIN12: now reaches U7.10 (B4Y)
- net DIN12: now also J4.09
- net DIN11: now reaches U7.11 (B3Y)
- net DIN11: now also J4.24
- net DIN10: now reaches U7.12 (B2Y)
- net DIN10: now also J4.10
- net DIN9: now reaches U7.13 (B1Y)
- net DIN9: now also J4.25
- net +3.3V: now reaches U7.14 (VCCB)
- net +3.3V: now also U10.14 (VCCB), U10.8 (OE), U5.14 (VCCB), U5.8 (OE), U6.14 (VCCB), U6.8 (OE), U7.8 (OE), U8.14 (VCCB), U8.8 (OE), U9.14 (VCCB), U9.8 (OE), C33.1, C34.1, C35.1, C36.1, C37.1, C38.1, C39.1, C40.1, C41.1, C42.1, C43.1
- net GND: now reaches U7.7 (GND)
- net GND: now also U10.7 (GND), U5.7 (GND), U6.7 (GND), U8.7 (GND), U9.7 (GND), C27.2, C28.2, C29.2, C30.2, C31.2, C33.2, C34.2, C35.2, C36.2, C37.2, C38.2, C39.2, C40.2, C41.2, C42.2, C43.2, J4.04, J4.08, J4.12, J4.19, J4.23, J4.27
- net DIN4: now reaches U5.10 (B4Y)
- net DIN4: now also J4.14
- net DIN3: now reaches U5.11 (B3Y)
- net DIN3: now also J4.29
- net DIN2: now reaches U5.12 (B2Y)
- net DIN2: now also J4.15
- net DIN1: now reaches U5.13 (B1Y)
- net DIN1: now also J4.30
- net DIN20: now reaches U9.10 (B4Y)
- net DIN20: now also J4.03
- net DIN19: now reaches U9.11 (B3Y)
- net DIN19: now also J4.18
- net DIN18: now reaches U9.12 (B2Y)
- net DIN18: now also J4.05
- net DIN17: now reaches U9.13 (B1Y)
- net DIN17: now also J4.20
- net DIN24: now reaches U10.10 (B4Y)
- net DIN24: now also J4.01
- net DIN23: now reaches U10.11 (B3Y)
- net DIN23: now also J4.16
- net DIN22: now reaches U10.12 (B2Y)
- net DIN22: now also J4.02
- net DIN21: now reaches U10.13 (B1Y)
- net DIN21: now also J4.17
- net DIN8: now reaches U6.10 (B4Y)
- net DIN8: now also J4.11
- net DIN7: now reaches U6.11 (B3Y)
- net DIN7: now also J4.26
- net DIN6: now reaches U6.12 (B2Y)
- net DIN6: now also J4.13
- net DIN5: now reaches U6.13 (B1Y)
- net DIN5: now also J4.28
- net DIN16: now reaches U8.10 (B4Y)
- net DIN16: now also J4.06
- net DIN15: now reaches U8.11 (B3Y)
- net DIN15: now also J4.21
- net DIN14: now reaches U8.12 (B2Y)
- net DIN14: now also J4.07
- net DIN13: now reaches U8.13 (B1Y)
- net DIN13: now also J4.22
Other:
- moved on the sheet: U10, U5, U6, U7, U8, U9

Commit message: Bus Connections to TB and TVS Diodes added
Parts:
- added D4, D5, D6: DFN3810-9L_824014885, Diode_SMD_Wurth:D_Wurth_WE-TVS-DFN3810-9L, symbol Diode_Wurth_WE-TVS:DFN3810-9L_824014885
Connections:
- net DIN1: now also D6.5
- net DIN10: now also D5.6
- net DIN11: now also D5.4
- net DIN12: now also D5.7
- net DIN13: now also D5.2
- net DIN14: now also D5.8
- net DIN15: now also D5.1
- net DIN16: now also D5.9
- net DIN17: now also D4.5
- net DIN18: now also D4.6
- net DIN19: now also D4.4
- net DIN2: now also D6.6
- net DIN20: now also D4.7
- net DIN21: now also D4.2
- net DIN22: now also D4.8
- net DIN23: now also D4.1
- net DIN24: now also D4.9
- net DIN3: now also D6.4
- net DIN4: now also D6.7
- net DIN5: now also D6.2
- net DIN6: now also D6.8
- net DIN7: now also D6.1
- net DIN8: now also D6.9
- net DIN9: now also D5.5
- net GND: now also D4.3 (GND), D5.3 (GND), D6.3 (GND)
Other:
- note added: "Level Shifters"
- note added: "Low Ct TVS Array"
- note added: "Terminal Block"
- moved on the sheet: C27, C28, C29, C30, C31, C32, C33, C34, C35, C36, C37, C38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

Commit message: Added EXT VREF, TRIG, ROTARY SWITCH, DAISY CHAIN CONNECTIONS etc
Parts:
- added D10, D11, D12, D8, D9: 0402_82307050029, Diode_SMD_Wurth:D_Wurth_WE-VE-ULC-0402, symbol 82307050029-TVS-Diode_Wurth_WE-VE-ULC:0402_82307050029
- added D7: LL4148, Diode_SMD:D_MiniMELF, symbol Diode:LL4148
- added J5, J6: 534269030, CONN03_534269030_MOL, symbol 534269030:534269030
- added J7: SSW-106-02-TM-S-RA, SSW-106-02-TM-S-RA:SAMTEC_SSW-106-02-TM-S-RA, symbol SSW-106-02-TM-S-RA:SSW-106-02-TM-S-RA
- added J8: 874370443, CONN_874370231-SD_04_MOL, symbol Molex-874370443:874370443
- added R39: 8K2, Resistor_SMD:R_0603_1608Metric_Pad0.98x0.95mm_HandSolder, symbol Device:R_Small
- added R40: 100K, Resistor_SMD:R_0603_1608Metric_Pad0.98x0.95mm_HandSolder, symbol Device:R_Small
Connections:
- net +3.3V: now also D12.2, J7.04, J8.3_1, J8.3_2
- net GND: now also D10.1, D11.1, D12.1, D8.1, D9.1, J5.3, J6.3, J7.03, R39.2, R40.1
- net VREF: now also D10.2, J7.06, J8.2_1, J8.2_2
- new net +5V: D11.2, J7.05, J8.4_2
- new net EXT_CHAIN: D7.2 (A), D8.2, D9.2, J5.1, J6.1, R39.1
- new net EXT_TRIG: D7.1 (K), J7.02, R40.2
- new net EXT_VREF: J7.01, J8.1_1, J8.1_2
Other:
- note added: "EXT CHAIN CONNECTOR 1"
- note added: "EXT CHAIN CONNECTOR 2"
- note added: "LEVEL SHIFTERS"
- note added: "LOGIC INPUTS"
- note added: "POWER AND TRIGGER ACCESS"
- note added: "TVS ARRAY"
- note added: "VREF SELECTOR CONNECTION TO ROTARY SWITCH"
- note removed: "Level Shifters"
- note removed: "Low Ct TVS Array"
- note removed: "Terminal Block"

Commit message: SOME AESTHETIC SCHEMATIC CHANGES
Other:
- moved on the sheet: D10, D11, D12, D7, D8, D9, J5, J6, J7, J8, R39, R40

Commit message: Connector for Front Panel Interface Added
Parts:
- removed D10: 0402_82307050029, Diode_SMD_Wurth:D_Wurth_WE-VE-ULC-0402, symbol 82307050029-TVS-Diode_Wurth_WE-VE-ULC:0402_82307050029
- removed J4: IPL1-115-01-X-D-RA-K, IPL1-115-01-X-D-RA-K:SAMTEC_IPL1-115-01-X-D-RA-K, symbol IPL1-115-01-X-D-RA-K:IPL1-115-01-X-D-RA-K
- removed J8: 874370443, CONN_874370231-SD_04_MOL, symbol Molex-874370443:874370443
- added J9: 612050235221, Connector_THT_Wurth:J_Wurth_WR-BHD_612050235221, symbol Connector_Wurth_WR-BHD:612050235221
Connections:
- net DIN1: now also J9.1
- net DIN10: now also J9.19
- net DIN11: now also J9.21
- net DIN12: now also J9.23
- net DIN13: now also J9.25
- net DIN14: now also J9.27
- net DIN15: now also J9.29
- net DIN16: now also J9.31
- net DIN17: now also J9.33
- net DIN18: now also J9.35
- net DIN19: now also J9.37
- net DIN2: now also J9.3
- net DIN20: now also J9.39
- net DIN21: now also J9.41
- net DIN22: now also J9.43
- net DIN23: now also J9.45
- net DIN24: now also J9.47
- net DIN3: now also J9.5
- net DIN4: now also J9.7
- net DIN5: now also J9.9
- net DIN6: now also J9.11
- net DIN7: now also J9.13
- net DIN8: now also J9.15
- net DIN9: now also J9.17
- net GND: now also J7.06, J9.10, J9.12, J9.14, J9.16, J9.18, J9.2, J9.20, J9.22, J9.24, J9.26, J9.28, J9.30, J9.32, J9.34, J9.36, J9.38, J9.4, J9.40, J9.42, J9.44, J9.46, J9.48, J9.49, J9.50, J9.6, J9.8
- net VREF: no longer J7.06
- net EXT_VREF renamed EXTVREF
Other:
- note removed: "LOGIC INPUTS"
- note removed: "VREF SELECTOR CONNECTION TO ROTARY SWITCH"
- moved on the sheet: D7, D8, D9, J5, J6, J7, R39, R40

Commit message: Clearing UP ERC Errors and Warnings
Parts:
- added C46: 100nF, Capacitor_SMD:C_0603_1608Metric_Pad1.08x0.95mm_HandSolder, symbol Device:C_Small
- added D10, D13: 0402_82307050029, 82307050029-TVS-Diode_Wurth_WE-VE-ULC:D_Wurth_WE-VE-ULC-0402, symbol 82307050029-TVS-Diode_Wurth_WE-VE-ULC:0402_82307050029
- D11, D12, D8, D9: footprint Diode_SMD_Wurth:D_Wurth_WE-VE-ULC-0402 -> 82307050029-TVS-Diode_Wurth_WE-VE-ULC:D_Wurth_WE-VE-ULC-0402
- J5, J6: footprint CONN03_534269030_MOL -> 534269030:CONN03_534269030_MOL
- J7: footprint SSW-106-02-TM-S-RA:SAMTEC_SSW-106-02-TM-S-RA -> SSW_106_02_TM_S_RA:SAMTEC_SSW-106-02-TM-S-RA
- U10, U5, U6, U7, U8, U9: footprint TSSOP_0104PWR_TEX -> TXU0104PWR:TSSOP_0104PWR_TEX
Connections:
- net +3.3V: now also C46.1
- net EXTVREF: now also D10.2
- net EXT_TRIG: now also D13.2
- net GND: now also C32.2, C46.2, D10.1, D13.1
- no-connect marks 0 -> 2

Commit message: Net Classes Added
Parts:
- renumbered C29 to C28, C31 to C29, C34 to C30, C35 to C31, C37 to C32, C39 to C33, C40 to C34, C41 to C35, C28 to C36, C30 to C37, C32 to C38, C33 to C39, C36 to C40, C38 to C41, C46 to C42, C42 to C43, C43 to C44, D11 to D10, D8 to D11, D6 to D13, D7 to D6, D10 to D7, D13 to D8, J7 to J3, J6 to J4, J9 to J6, R39 to R43, R40 to R44
Other:
- note added: "Logic Input Connector"
