File: LogicAnalyzer_RP2350/LogicAnalyzer_RP2350/LevelShifters.kicad_sch (KiCad schematic)
At the start: 40 parts, among them J3 SSW-106-02-TM-S-RA, J4 534269030, J5 534269030, J6 612050235221, U10 TXU0104PWR, U5 TXU0104PWR, U6 TXU0104PWR, U7 TXU0104PWR, U8 TXU0104PWR, U9 TXU0104PWR

Commit message: Added Missing 3D Models
Other:
- moved on the sheet: C27, C28, C29, C30, C31, C32, C33, C34, C35, C36, C37, C38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

Commit message: TVS Swapped to more routing friendly, adjusting the Positions of TVs and Connectors
Parts:
- removed D13, D4, D5: DFN3810-9L_824014885, Diode_SMD_Wurth:D_Wurth_WE-TVS-DFN3810-9L, symbol Diode_Wurth_WE-TVS:DFN3810-9L_824014885
- added D13, D14, D15, D16, D17, D18, D19, D20, D21, D22, D4, D5: SOT563_82400152, Diode_SMD_Wurth:D_Wurth_WE-TVS-SOT563, symbol Diode_Wurth_WE-TVS:SOT563_82400152
Connections:
- net +5V: now also D13.5 (VDD), D14.5 (VDD), D15.5 (VDD), D16.5 (VDD), D17.5 (VDD), D18.5 (VDD), D19.5 (VDD), D20.5 (VDD), D21.5 (VDD), D22.5 (VDD), D4.5 (VDD), D5.5 (VDD)
- net D1: now also U5.5 (A4); no longer U5.2 (A1)
- net D10: now also U7.4 (A3); no longer U7.3 (A2)
- net D11: now also U7.3 (A2); no longer U7.4 (A3)
- net D12: now also U7.2 (A1); no longer U7.5 (A4)
- net D13: now also U8.5 (A4); no longer U8.2 (A1)
- net D14: now also U8.4 (A3); no longer U8.3 (A2)
- net D15: now also U8.3 (A2); no longer U8.4 (A3)
- net D16: now also U8.2 (A1); no longer U8.5 (A4)
- net D17: now also U9.5 (A4); no longer U9.2 (A1)
- net D18: now also U9.4 (A3); no longer U9.3 (A2)
- net D19: now also U9.3 (A2); no longer U9.4 (A3)
- net D2: now also U5.4 (A3); no longer U5.3 (A2)
- net D20: now also U9.2 (A1); no longer U9.5 (A4)
- net D21: now also U10.5 (A4); no longer U10.2 (A1)
- net D22: now also U10.4 (A3); no longer U10.3 (A2)
- net D23: now also U10.3 (A2); no longer U10.4 (A3)
- net D24: now also U10.2 (A1); no longer U10.5 (A4)
- net D3: now also U5.3 (A2); no longer U5.4 (A3)
- net D4: now also U5.2 (A1); no longer U5.5 (A4)
- net D5: now also U6.5 (A4); no longer U6.2 (A1)
- net D6: now also U6.4 (A3); no longer U6.3 (A2)
- net D7: now also U6.3 (A2); no longer U6.4 (A3)
- net D8: now also U6.2 (A1); no longer U6.5 (A4)
- net D9: now also U7.5 (A4); no longer U7.2 (A1)
- net DIN1: now also U5.10 (B4Y), D4.3 (I/O2); no longer J6.1, U5.13 (B1Y)
- net DIN10: now also U7.11 (B3Y), D15.1 (I/O1); no longer J6.19, U7.12 (B2Y)
- net DIN11: now also U7.12 (B2Y), D16.3 (I/O2); no longer J6.21, U7.11 (B3Y)
- net DIN12: now also U7.13 (B1Y), D16.1 (I/O1); no longer J6.23, U7.10 (B4Y)
- net DIN13: now also U8.10 (B4Y), D17.3 (I/O2); no longer J6.25, U8.13 (B1Y)
- net DIN14: now also U8.11 (B3Y), D17.1 (I/O1); no longer J6.27, U8.12 (B2Y)
- net DIN15: now also U8.12 (B2Y), D18.3 (I/O2); no longer J6.29, U8.11 (B3Y)
- net DIN16: now also U8.13 (B1Y), D18.1 (I/O1); no longer J6.31, U8.10 (B4Y)
- net DIN17: now also U9.10 (B4Y), D19.3 (I/O2); no longer J6.33, U9.13 (B1Y)
- net DIN18: now also U9.11 (B3Y), D19.1 (I/O1); no longer J6.35, U9.12 (B2Y)
- net DIN19: now also U9.12 (B2Y), D20.3 (I/O2); no longer J6.37, U9.11 (B3Y)
- net DIN2: now also U5.11 (B3Y), D4.1 (I/O1); no longer J6.3, U5.12 (B2Y)
- net DIN20: now also U9.13 (B1Y), D20.1 (I/O1); no longer J6.39, U9.10 (B4Y)
- net DIN21: now also U10.10 (B4Y), D21.3 (I/O2); no longer J6.41, U10.13 (B1Y)
- net DIN22: now also U10.11 (B3Y), D21.1 (I/O1); no longer J6.43, U10.12 (B2Y)
- net DIN23: now also U10.12 (B2Y), D22.3 (I/O2); no longer J6.45, U10.11 (B3Y)
- net DIN24: now also U10.13 (B1Y), D22.1 (I/O1); no longer J6.47, U10.10 (B4Y)
- net DIN3: now also U5.12 (B2Y), D5.3 (I/O2); no longer J6.5, U5.11 (B3Y)
- net DIN4: now also U5.13 (B1Y), D5.1 (I/O1); no longer J6.7, U5.10 (B4Y)
- net DIN5: now also U6.10 (B4Y), D13.3 (I/O2); no longer J6.9, U6.13 (B1Y)
- net DIN6: now also U6.11 (B3Y), D13.1 (I/O1); no longer J6.11, U6.12 (B2Y)
- net DIN7: now also U6.12 (B2Y), D14.3 (I/O2); no longer J6.13, U6.11 (B3Y)
- net DIN8: now also U6.13 (B1Y), D14.1 (I/O1); no longer J6.15, U6.10 (B4Y)
- net DIN9: now also U7.10 (B4Y), D15.3 (I/O2); no longer J6.17, U7.13 (B1Y)
- net GND: now also D13.2 (GND), D14.2 (GND), D15.2 (GND), D16.2 (GND), D17.2 (GND), D18.2 (GND), D19.2 (GND), D20.2 (GND), D21.2 (GND), D22.2 (GND), D4.2 (GND), D5.2 (GND)
- new net DI1: D4.4 (I/O4), J6.47
- new net DI10: D15.6 (I/O3), J6.29
- new net DI11: D16.4 (I/O4), J6.27
- new net DI12: D16.6 (I/O3), J6.25
- new net DI13: D17.4 (I/O4), J6.23
- new net DI14: D17.6 (I/O3), J6.21
- new net DI15: D18.4 (I/O4), J6.19
- new net DI16: D18.6 (I/O3), J6.17
- new net DI17: D19.4 (I/O4), J6.15
- new net DI18: D19.6 (I/O3), J6.13
- new net DI19: D20.4 (I/O4), J6.11
- new net DI2: D4.6 (I/O3), J6.45
- new net DI20: D20.6 (I/O3), J6.9
- new net DI21: D21.4 (I/O4), J6.7
- new net DI22: D21.6 (I/O3), J6.5
- new net DI23: D22.4 (I/O4), J6.3
- new net DI24: D22.6 (I/O3), J6.1
- new net DI3: D5.4 (I/O4), J6.43
- new net DI4: D5.6 (I/O3), J6.41
- new net DI5: D13.4 (I/O4), J6.39
- new net DI6: D13.6 (I/O3), J6.37
- new net DI7: D14.4 (I/O4), J6.35
- new net DI8: D14.6 (I/O3), J6.33
- new net DI9: D15.4 (I/O4), J6.31
Other:
- moved on the sheet: D10, D11, D12, D6, D7, D8, D9, J3, J4, J5, J6, R43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
