File: LogicAnalyzer_RP2350/LogicAnalyzer_RP2350/LogicAnalyzer_RP2350.kicad_pcb (KiCad board)
At the start: 4 copper layers, 0 parts

Commit message: Added Missing 3D Models
Parts:
- added A1: 9774050151R, Assembly_SMD_Wurth:A_Wurth_WA-SMSI_9774050151R, F.Cu at (147.6, 127.4)
- added A2: 9774050151R, Assembly_SMD_Wurth:A_Wurth_WA-SMSI_9774050151R, F.Cu at (147.6, 135.0)
- added A3: 9774050151R, Assembly_SMD_Wurth:A_Wurth_WA-SMSI_9774050151R, F.Cu at (147.6, 142.5)
- added A4: 9774050151R, Assembly_SMD_Wurth:A_Wurth_WA-SMSI_9774050151R, F.Cu at (147.6, 150.1)
- added C1: 10nF/50V, Capacitor_SMD:C_0805_2012Metric_Pad1.18x1.45mm_HandSolder, F.Cu at (157.1, 99.8)
- added C10: 4.7uF, Capacitor_SMD:C_0603_1608Metric_Pad1.08x0.95mm_HandSolder, F.Cu at (146.0, 70.8)
- added C11: 4.7uF, Capacitor_SMD:C_0603_1608Metric_Pad1.08x0.95mm_HandSolder, F.Cu at (146.0, 73.3)
- added C12: 15pF, Capacitor_SMD:C_0603_1608Metric_Pad1.08x0.95mm_HandSolder, F.Cu at (146.0, 75.8)
- added C13: 15pF, Capacitor_SMD:C_0603_1608Metric_Pad1.08x0.95mm_HandSolder, F.Cu at (146.0, 78.3)
- added C14: 100nF, Capacitor_SMD:C_0603_1608Metric_Pad1.08x0.95mm_HandSolder, F.Cu at (146.0, 80.8)
- added C15: 4.7uF, Capacitor_SMD:C_0603_1608Metric_Pad1.08x0.95mm_HandSolder, F.Cu at (146.0, 83.3)
- added C16: 4.7uF, Capacitor_SMD:C_0603_1608Metric_Pad1.08x0.95mm_HandSolder, F.Cu at (146.0, 85.8)
- added C17: 100nF, Capacitor_SMD:C_0603_1608Metric_Pad1.08x0.95mm_HandSolder, F.Cu at (150.4, 65.8)
- added C18: 100nF, Capacitor_SMD:C_0603_1608Metric_Pad1.08x0.95mm_HandSolder, F.Cu at (150.4, 68.3)
- added C19: 100nF, Capacitor_SMD:C_0603_1608Metric_Pad1.08x0.95mm_HandSolder, F.Cu at (150.4, 70.8)
- added C2: 100nF, Capacitor_SMD:C_0805_2012Metric_Pad1.18x1.45mm_HandSolder, F.Cu at (157.1, 102.9)
- added C20: 100nF, Capacitor_SMD:C_0603_1608Metric_Pad1.08x0.95mm_HandSolder, F.Cu at (150.4, 73.3)
- added C21: 100nF, Capacitor_SMD:C_0603_1608Metric_Pad1.08x0.95mm_HandSolder, F.Cu at (150.4, 75.8)
- added C22: 100nF, Capacitor_SMD:C_0603_1608Metric_Pad1.08x0.95mm_HandSolder, F.Cu at (150.4, 78.3)
- added C23: 100nF, Capacitor_SMD:C_0603_1608Metric_Pad1.08x0.95mm_HandSolder, F.Cu at (150.4, 80.8)
- added C24: 100nF, Capacitor_SMD:C_0603_1608Metric_Pad1.08x0.95mm_HandSolder, F.Cu at (150.4, 83.3)
- added C25: 100nF, Capacitor_SMD:C_0603_1608Metric_Pad1.08x0.95mm_HandSolder, F.Cu at (150.4, 85.8)
- added C26: 100nF, Capacitor_SMD:C_0603_1608Metric_Pad1.08x0.95mm_HandSolder, F.Cu at (154.7, 65.8)
- added C27: 100nF, Capacitor_SMD:C_0603_1608Metric_Pad1.08x0.95mm_HandSolder, F.Cu at (120.9, 118.6)
- added C28: 100nF, Capacitor_SMD:C_0603_1608Metric_Pad1.08x0.95mm_HandSolder, F.Cu at (120.9, 121.1)
- added C29: 100nF, Capacitor_SMD:C_0603_1608Metric_Pad1.08x0.95mm_HandSolder, F.Cu at (120.9, 123.6)
- added C3: 4.7 uF, Capacitor_SMD_Wurth:CP_Wurth_WCAP-ASLI-D4L5.5, F.Cu at (163.6, 101.5)
- added C30: 100nF, Capacitor_SMD:C_0603_1608Metric_Pad1.08x0.95mm_HandSolder, F.Cu at (120.9, 126.1)
- added C31: 100nF, Capacitor_SMD:C_0603_1608Metric_Pad1.08x0.95mm_HandSolder, F.Cu at (120.9, 128.7)
- added C32: 100nF, Capacitor_SMD:C_0603_1608Metric_Pad1.08x0.95mm_HandSolder, F.Cu at (125.2, 118.6)
- added C33: 100nF, Capacitor_SMD:C_0603_1608Metric_Pad1.08x0.95mm_HandSolder, F.Cu at (125.2, 121.1)
- added C34: 100nF, Capacitor_SMD:C_0603_1608Metric_Pad1.08x0.95mm_HandSolder, F.Cu at (125.2, 123.6)
- added C35: 100nF, Capacitor_SMD:C_0603_1608Metric_Pad1.08x0.95mm_HandSolder, F.Cu at (125.2, 126.1)
- added C36: 100nF, Capacitor_SMD:C_0603_1608Metric_Pad1.08x0.95mm_HandSolder, F.Cu at (125.2, 128.7)
- added C37: 100nF, Capacitor_SMD:C_0603_1608Metric_Pad1.08x0.95mm_HandSolder, F.Cu at (129.6, 118.6)
- added C38: 100nF, Capacitor_SMD:C_0603_1608Metric_Pad1.08x0.95mm_HandSolder, F.Cu at (129.6, 121.1)
- added C39: 100nF, Capacitor_SMD:C_0603_1608Metric_Pad1.08x0.95mm_HandSolder, F.Cu at (129.6, 123.6)
- added C4: 10uF, Capacitor_SMD:C_0805_2012Metric_Pad1.18x1.45mm_HandSolder, F.Cu at (157.1, 105.9)
- added C40: 100nF, Capacitor_SMD:C_0603_1608Metric_Pad1.08x0.95mm_HandSolder, F.Cu at (129.6, 126.1)
- added C41: 100nF, Capacitor_SMD:C_0603_1608Metric_Pad1.08x0.95mm_HandSolder, F.Cu at (129.6, 128.7)
- added C42: 100nF, Capacitor_SMD:C_0603_1608Metric_Pad1.08x0.95mm_HandSolder, F.Cu at (133.9, 118.6)
- added C43: 100nF, Capacitor_SMD:C_0603_1608Metric_Pad1.08x0.95mm_HandSolder, F.Cu at (133.9, 121.1)
- added C44: 100nF, Capacitor_SMD:C_0603_1608Metric_Pad1.08x0.95mm_HandSolder, F.Cu at (133.9, 123.6)
- added C45: 100nF, Capacitor_SMD:C_0603_1608Metric_Pad1.08x0.95mm_HandSolder, F.Cu at (166.2, 132.5)
- added C46: 1uF, Capacitor_SMD:C_0603_1608Metric_Pad1.08x0.95mm_HandSolder, F.Cu at (166.2, 135.0)
- added C5: 100nF, Capacitor_SMD:C_0603_1608Metric_Pad1.08x0.95mm_HandSolder, F.Cu at (146.0, 99.6)
- added C6: 10uF, Capacitor_SMD:C_0805_2012Metric_Pad1.18x1.45mm_HandSolder, F.Cu at (157.1, 108.9)
- added C7: 10uF/50V, Capacitor_SMD:C_0805_2012Metric_Pad1.18x1.45mm_HandSolder, F.Cu at (157.1, 111.9)
- added C8: 100nF, Capacitor_SMD:C_0603_1608Metric_Pad1.08x0.95mm_HandSolder, F.Cu at (146.0, 65.8)
- added C9: 4.7uF, Capacitor_SMD:C_0603_1608Metric_Pad1.08x0.95mm_HandSolder, F.Cu at (146.0, 68.3)
- added D1: 0402_82307050029, 82307050029-TVS-Diode_Wurth_WE-VE-ULC:D_Wurth_WE-VE-ULC-0402, F.Cu at (165.5, 110.3)
- added D10: 0402_82307050029, 82307050029-TVS-Diode_Wurth_WE-VE-ULC:D_Wurth_WE-VE-ULC-0402, F.Cu at (129.4, 98.7)
- added D11: 0402_82307050029, 82307050029-TVS-Diode_Wurth_WE-VE-ULC:D_Wurth_WE-VE-ULC-0402, F.Cu at (129.4, 100.9)
- added D12: 0402_82307050029, 82307050029-TVS-Diode_Wurth_WE-VE-ULC:D_Wurth_WE-VE-ULC-0402, F.Cu at (129.4, 103.2)
- added D13: DFN3810-9L_824014885, Diode_SMD_Wurth:D_Wurth_WE-TVS-DFN3810-9L, F.Cu at (139.0, 93.5)
- added D2: SOT23-5L_824011, Diode_SMD_Wurth:D_Wurth_WE-TVS-SOT23-5L, F.Cu at (162.2, 106.9)
- added D3: LED_Blue, LED_SMD:LED_0603_1608Metric_Pad1.05x0.95mm_HandSolder, F.Cu at (173.9, 93.9)
- added D4: DFN3810-9L_824014885, Diode_SMD_Wurth:D_Wurth_WE-TVS-DFN3810-9L, F.Cu at (132.6, 93.5)
- added D5: DFN3810-9L_824014885, Diode_SMD_Wurth:D_Wurth_WE-TVS-DFN3810-9L, F.Cu at (135.8, 93.5)
- added D6: LL4148, Diode_SMD:D_MiniMELF, F.Cu at (134.1, 97.8)
- added D7: 0402_82307050029, 82307050029-TVS-Diode_Wurth_WE-VE-ULC:D_Wurth_WE-VE-ULC-0402, F.Cu at (129.4, 92.0)
- added D8: 0402_82307050029, 82307050029-TVS-Diode_Wurth_WE-VE-ULC:D_Wurth_WE-VE-ULC-0402, F.Cu at (129.4, 94.2)
- added D9: 0402_82307050029, 82307050029-TVS-Diode_Wurth_WE-VE-ULC:D_Wurth_WE-VE-ULC-0402, F.Cu at (129.4, 96.4)
- added FID1: Fiducial, Fiducial:Fiducial_1mm_Mask2mm, F.Cu at (153.2, 125.4)
- added FID2: Fiducial, Fiducial:Fiducial_1mm_Mask2mm, F.Cu at (153.2, 129.0)
- added FID3: Fiducial, Fiducial:Fiducial_1mm_Mask2mm, F.Cu at (156.7, 125.4)
- added FID4: Fiducial, Fiducial:Fiducial_1mm_Mask2mm, F.Cu at (156.7, 129.0)
- added FID5: Fiducial, Fiducial:Fiducial_1mm_Mask2mm, F.Cu at (160.3, 125.4)
- added FID6: Fiducial, Fiducial:Fiducial_1mm_Mask2mm, F.Cu at (160.3, 129.0)
- added J1: 2169890001, USBC_Molex_2169890001:216989-0001_MOL, F.Cu at (151.6, 105.7)
- added J2: SM03B-SRSS-TB, Connector_JST:JST_SH_SM03B-SRSS-TB_1x03-1MP_P1.00mm_Horizontal, F.Cu at (167.8, 90.9)
- added J3: SSW-106-02-TM-S-RA, SSW_106_02_TM_S_RA:SAMTEC_SSW-106-02-TM-S-RA, F.Cu at (133.7, 115.9)
- added J4: 534269030, 534269030:CONN03_534269030_MOL, F.Cu at (133.6, 67.9)
- added J5: 534269030, 534269030:CONN03_534269030_MOL, F.Cu at (133.6, 81.0)
- added J6: 612050235221, Connector_THT_Wurth:J_Wurth_WR-BHD_612050235221, F.Cu at (104.7, 70.7)
- added J7: 533984003, Molex-533984003:CONN_533980002-SD_03_MOL, F.Cu at (174.2, 148.8)
- added J8: 2035571207, Molex-2035571207:CONN_2035570000-SD_12_MOL, F.Cu at (172.3, 128.1)
- added L1: 167 nH, Inductor_SMD_Wurth:L_Wurth_WE-CNSW-HF-0805, F.Cu at (150.3, 116.0)
- added L2: BLM18PG221SN1D, Ferrite-BLM18PG221SN1D:IND_BLM18_0603_MUR, F.Cu at (150.3, 118.7)
- added L3: AOTA-B201610S3R3-101-T, ABRACON AOTA-B201610S3R3-101-T:AOTAB201610S3R3101T, F.Cu at (173.0, 80.5)
- added R1: 5K6, Resistor_SMD:R_0603_1608Metric_Pad0.98x0.95mm_HandSolder, F.Cu at (146.0, 102.1)
- added R10: 10K, Resistor_SMD:R_0603_1608Metric_Pad0.98x0.95mm_HandSolder, F.Cu at (154.7, 73.3)
- added R11: 100R, Resistor_SMD:R_0603_1608Metric_Pad0.98x0.95mm_HandSolder, F.Cu at (154.7, 75.8)
- added R12: 100R, Resistor_SMD:R_0603_1608Metric_Pad0.98x0.95mm_HandSolder, F.Cu at (154.7, 78.3)
- added R13: 33R, Resistor_SMD:R_0603_1608Metric_Pad0.98x0.95mm_HandSolder, F.Cu at (154.7, 80.8)
- added R14: 1K, Resistor_SMD:R_0603_1608Metric_Pad0.98x0.95mm_HandSolder, F.Cu at (154.7, 83.3)
- added R15: 27R, Resistor_SMD:R_0603_1608Metric_Pad0.98x0.95mm_HandSolder, F.Cu at (154.7, 85.8)
- added R16: 27R, Resistor_SMD:R_0603_1608Metric_Pad0.98x0.95mm_HandSolder, F.Cu at (159.1, 65.8)
- added R17: 33R, Resistor_SMD:R_0603_1608Metric_Pad0.98x0.95mm_HandSolder, F.Cu at (159.1, 68.3)
- added R18: 470R, Resistor_SMD:R_0603_1608Metric_Pad0.98x0.95mm_HandSolder, F.Cu at (159.1, 70.8)
- added R19: 33R, Resistor_SMD:R_0603_1608Metric_Pad0.98x0.95mm_HandSolder, F.Cu at (159.1, 73.3)
- added R2: 10K, Resistor_SMD:R_0603_1608Metric_Pad0.98x0.95mm_HandSolder, F.Cu at (146.0, 104.6)
- added R20: 33R, Resistor_SMD:R_0603_1608Metric_Pad0.98x0.95mm_HandSolder, F.Cu at (159.1, 75.8)
- added R21: 33R, Resistor_SMD:R_0603_1608Metric_Pad0.98x0.95mm_HandSolder, F.Cu at (159.1, 78.3)
- added R22: 33R, Resistor_SMD:R_0603_1608Metric_Pad0.98x0.95mm_HandSolder, F.Cu at (159.1, 80.8)
- added R23: 33R, Resistor_SMD:R_0603_1608Metric_Pad0.98x0.95mm_HandSolder, F.Cu at (159.1, 83.3)
- added R24: 33R, Resistor_SMD:R_0603_1608Metric_Pad0.98x0.95mm_HandSolder, F.Cu at (159.1, 85.8)
- added R25: 33R, Resistor_SMD:R_0603_1608Metric_Pad0.98x0.95mm_HandSolder, F.Cu at (163.4, 65.8)
- added R26: 33R, Resistor_SMD:R_0603_1608Metric_Pad0.98x0.95mm_HandSolder, F.Cu at (163.4, 68.3)
- added R27: 33R, Resistor_SMD:R_0603_1608Metric_Pad0.98x0.95mm_HandSolder, F.Cu at (163.4, 70.8)
- added R28: 33R, Resistor_SMD:R_0603_1608Metric_Pad0.98x0.95mm_HandSolder, F.Cu at (163.4, 73.3)
- added R29: 33R, Resistor_SMD:R_0603_1608Metric_Pad0.98x0.95mm_HandSolder, F.Cu at (163.4, 75.8)
- added R3: 5K1, Resistor_SMD:R_0603_1608Metric_Pad0.98x0.95mm_HandSolder, F.Cu at (146.0, 107.1)
- added R30: 33R, Resistor_SMD:R_0603_1608Metric_Pad0.98x0.95mm_HandSolder, F.Cu at (163.4, 78.3)
- added R31: 33R, Resistor_SMD:R_0603_1608Metric_Pad0.98x0.95mm_HandSolder, F.Cu at (163.4, 80.8)
- added R32: 33R, Resistor_SMD:R_0603_1608Metric_Pad0.98x0.95mm_HandSolder, F.Cu at (163.4, 83.3)
- added R33: 33R, Resistor_SMD:R_0603_1608Metric_Pad0.98x0.95mm_HandSolder, F.Cu at (163.4, 85.8)
- added R34: 33R, Resistor_SMD:R_0603_1608Metric_Pad0.98x0.95mm_HandSolder, F.Cu at (167.8, 65.8)
- added R35: 33R, Resistor_SMD:R_0603_1608Metric_Pad0.98x0.95mm_HandSolder, F.Cu at (167.8, 68.3)
- added R36: 33R, Resistor_SMD:R_0603_1608Metric_Pad0.98x0.95mm_HandSolder, F.Cu at (167.8, 70.8)
- added R37: 33R, Resistor_SMD:R_0603_1608Metric_Pad0.98x0.95mm_HandSolder, F.Cu at (167.8, 73.3)
- added R38: 33R, Resistor_SMD:R_0603_1608Metric_Pad0.98x0.95mm_HandSolder, F.Cu at (167.8, 75.8)
- added R39: 33R, Resistor_SMD:R_0603_1608Metric_Pad0.98x0.95mm_HandSolder, F.Cu at (167.8, 78.3)
- added R4: 5K1, Resistor_SMD:R_0603_1608Metric_Pad0.98x0.95mm_HandSolder, F.Cu at (146.0, 109.6)
- added R40: 33R, Resistor_SMD:R_0603_1608Metric_Pad0.98x0.95mm_HandSolder, F.Cu at (167.8, 80.8)
- added R41: 33R, Resistor_SMD:R_0603_1608Metric_Pad0.98x0.95mm_HandSolder, F.Cu at (167.8, 83.3)
- added R42: 33R, Resistor_SMD:R_0603_1608Metric_Pad0.98x0.95mm_HandSolder, F.Cu at (167.8, 85.8)
- added R43: 8K2, Resistor_SMD:R_0603_1608Metric_Pad0.98x0.95mm_HandSolder, F.Cu at (133.9, 126.1)
- added R44: 100K, Resistor_SMD:R_0603_1608Metric_Pad0.98x0.95mm_HandSolder, F.Cu at (133.9, 128.7)
- added R45: 4.7K, Resistor_SMD:R_0603_1608Metric_Pad0.98x0.95mm_HandSolder, F.Cu at (166.2, 137.5)
- added R46: 4.7K, Resistor_SMD:R_0603_1608Metric_Pad0.98x0.95mm_HandSolder, F.Cu at (166.2, 140.0)
- added R47: 100R, Resistor_SMD:R_0603_1608Metric_Pad0.98x0.95mm_HandSolder, F.Cu at (166.2, 142.5)
- added R48: 4.7K, Resistor_SMD:R_0603_1608Metric_Pad0.98x0.95mm_HandSolder, F.Cu at (166.2, 145.0)
- added R49: 4.7K, Resistor_SMD:R_0603_1608Metric_Pad0.98x0.95mm_HandSolder, F.Cu at (166.2, 147.5)
- added R5: 100K, Resistor_SMD:R_0603_1608Metric_Pad0.98x0.95mm_HandSolder, F.Cu at (146.0, 112.1)
- added R6: 100K, Resistor_SMD:R_0603_1608Metric_Pad0.98x0.95mm_HandSolder, F.Cu at (146.0, 114.7)
- added R7: 25K 1%, Resistor_SMD:R_0603_1608Metric_Pad0.98x0.95mm_HandSolder, F.Cu at (146.0, 117.2)
- added R8: 10K, Resistor_SMD:R_0603_1608Metric_Pad0.98x0.95mm_HandSolder, F.Cu at (154.7, 68.3)
- added R9: 1K, Resistor_SMD:R_0603_1608Metric_Pad0.98x0.95mm_HandSolder, F.Cu at (154.7, 70.8)
- added SW1: SW_MEC_5G, SKRPABE010:SW4_SKRPABE010_ALPS, F.Cu at (174.6, 67.9)
- added SW2: SW_MEC_5G, SKRPABE010:SW4_SKRPABE010_ALPS, F.Cu at (174.6, 74.8)
- added U1: NCP1117ST33T3G, NCP1117:SOT230P700X180-4N, F.Cu at (159.5, 117.5)
- added U10: TXU0104PWR, TXU0104PWR:TSSOP_0104PWR_TEX, F.Cu at (123.2, 101.7)
- added U11: ATtiny3216-S, Package_SO:SOIC-20W_7.5x12.8mm_P1.27mm, F.Cu at (174.9, 138.5)
- added U2: TPS2552DRVR-1, TPS2552DRVR:DRV6_1P6X1, F.Cu at (161.7, 111.0)
- added U3: W25Q128JVS, Package_SO:SOIC-8_5.3x5.3mm_P1.27mm, F.Cu at (149.0, 90.6)
- added U4: RP2350A, Package_DFN_QFN:QFN-60-1EP_7x7mm_P0.4mm_EP3.4x3.4mm_ThermalVias, F.Cu at (159.2, 91.7)
- added U5: TXU0104PWR, TXU0104PWR:TSSOP_0104PWR_TEX, F.Cu at (123.2, 67.9)
- added U6: TXU0104PWR, TXU0104PWR:TSSOP_0104PWR_TEX, F.Cu at (123.2, 74.6)
- added U7: TXU0104PWR, TXU0104PWR:TSSOP_0104PWR_TEX, F.Cu at (123.2, 81.4)
- added U8: TXU0104PWR, TXU0104PWR:TSSOP_0104PWR_TEX, F.Cu at (123.2, 88.2)
- added U9: TXU0104PWR, TXU0104PWR:TSSOP_0104PWR_TEX, F.Cu at (123.2, 94.9)
- added Y1: 12Mhz, ABM8-272-T3:ABM8-272-T3_ABR, F.Cu at (175.5, 90.0)
