File: LogicAnalyzer_RP2350/LogicAnalyzer_RP2350/LogicAnalyzer_RP2350.kicad_pcb (KiCad board)
At the start: 4 copper layers, 143 parts, among them J1 2169890001, J2 SM03B-SRSS-TB, J3 SSW-106-02-TM-S-RA, J4 534269030, J5 534269030, J6 612050235221, J7 533984003, J8 2035571207, SW1 SW_MEC_5G, SW2 SW_MEC_5G, U1 NCP1117ST33T3G, U10 TXU0104PWR, U11 ATtiny3216-S, U2 TPS2552DRVR-1, U3 W25Q128JVS, U4 RP2350A, U5 TXU0104PWR, U6 TXU0104PWR, U7 TXU0104PWR, U8 TXU0104PWR, U9 TXU0104PWR, Y1 12Mhz

Commit message: Some Initial Rough placement
Parts:
- A1, A2: moved to B.Cu
- moved D6 203.8 mm to (337.8, 92.4)
- moved L2 203.8 mm to (354.0, 113.2)
- moved C26 203.8 mm to (358.5, 60.3)
- moved C27 203.8 mm to (324.6, 113.2)
- moved C28 203.8 mm to (324.6, 115.7)
- moved C29 203.8 mm to (324.6, 118.2)
- moved C30 203.8 mm to (324.6, 120.7)
- moved C31 203.8 mm to (324.6, 123.2)
- moved C37 203.8 mm to (333.3, 113.2)
- moved C38 203.8 mm to (333.3, 115.7)
- moved C39 203.8 mm to (333.3, 118.2)
- moved C40 203.8 mm to (333.3, 120.7)
- moved C41 203.8 mm to (333.3, 123.2)
- moved C45 203.8 mm to (370.0, 127.0)
- moved C46 203.8 mm to (370.0, 129.5)
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Other:
- board outline added: 130.5 x 80.5 mm

Commit message: Some Cleanup and Replacaing USB C connector
Parts:
- A1, A2: moved to F.Cu
- J1: value 2169890001 -> USB_C_Receptacle_USB2.0_16P; footprint USBC_Molex_2169890001:216989-0001_MOL -> Connector_USB:USB_C_Receptacle_GCT_USB4105-xx-A_16P_TopMnt_Horizontal
- moved C26 159.6 mm to (200.0, 41.8)
- moved C27 159.6 mm to (166.1, 94.7)
- moved C28 159.6 mm to (166.1, 97.2)
- moved C29 159.6 mm to (166.1, 99.7)
- moved C30 159.6 mm to (166.1, 102.2)
- moved C31 159.6 mm to (166.1, 104.7)
- moved C45 159.6 mm to (211.5, 108.5)
- moved C46 159.6 mm to (211.5, 111.1)
- moved D1 159.6 mm to (210.7, 86.3)
- moved D10 159.6 mm to (174.6, 74.8)
- moved D11 159.6 mm to (174.6, 77.0)
- moved D12 159.6 mm to (174.6, 79.2)
- moved D6 159.6 mm to (179.3, 73.9)
- moved D7 159.6 mm to (174.6, 68.0)
- moved D8 159.6 mm to (174.6, 70.3)
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Other:
- board outline removed

Commit message: Few more placement Corrections
Parts:
- C10, C11, C12, C13, C15, C16, C21, C22, C25, C8, C9: footprint Capacitor_SMD:C_0603_1608Metric_Pad1.08x0.95mm_HandSolder -> Capacitor_SMD:C_0402_1005Metric_Pad0.74x0.62mm_HandSolder
- C14, C17, C18, C19, C20, C23, C24, C26: footprint Capacitor_SMD:C_0603_1608Metric_Pad1.08x0.95mm_HandSolder -> Capacitor_SMD:C_0402_1005Metric_Pad0.74x0.62mm_HandSolder; moved to B.Cu
- R15, R16, R19, R20, R21, R22, R23, R24, R25, R26, R27, R28, R29, R30, R31, R32, R33, R34, R35, R36, R37, R38, R39, R40, R41, R42: footprint Resistor_SMD:R_0603_1608Metric_Pad0.98x0.95mm_HandSolder -> Resistor_SMD:R_0402_1005Metric_Pad0.72x0.64mm_HandSolder
- moved A1 172.1 mm to (365.0, 105.7)
- moved A2 172.1 mm to (365.0, 113.3)
- moved A3 172.1 mm to (365.0, 120.8)
- moved A4 172.1 mm to (365.0, 128.4)
- moved C3 172.1 mm to (381.0, 79.8)
- moved C32 172.1 mm to (342.6, 96.9)
- moved C33 172.1 mm to (342.6, 99.4)
- moved C34 172.1 mm to (342.6, 101.9)
- moved C35 172.1 mm to (342.6, 104.5)
- moved C36 172.1 mm to (342.6, 107.0)
- moved D2 172.1 mm to (379.5, 85.2)
- moved J1 172.1 mm to (406.7, 88.6)
- moved J2 172.1 mm to (385.1, 69.2)
- moved J4 172.1 mm to (350.9, 46.2)
- moved J5 172.1 mm to (350.9, 59.4)
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
Commit message: PCB outline Defined 100X80
Parts:
- A1, A2, A3, A4: moved to B.Cu
- R14, R17: footprint Resistor_SMD:R_0603_1608Metric_Pad0.98x0.95mm_HandSolder -> Resistor_SMD:R_0402_1005Metric_Pad0.72x0.64mm_HandSolder
- moved A3 253.4 mm to (119.5, 58.0), turned to 180 degrees
- moved SW1 253.3 mm to (140.5, 77.4)
- moved C4 249.2 mm to (125.6, 71.6), turned to -90 degrees
- moved J1 248.5 mm to (160.1, 57.6), turned to 180 degrees
- moved U1 247.7 mm to (130.3, 71.4), turned to -90 degrees
- moved A1 245.6 mm to (119.5, 113.8), turned to 180 degrees
- moved U2 243.9 mm to (136.6, 63.1), turned to -90 degrees
- moved C6 239.9 mm to (135.1, 71.6), turned to 90 degrees
- moved C7 239.3 mm to (137.1, 59.4), turned to 180 degrees
- moved C3 239.3 mm to (142.3, 61.6), turned to 90 degrees
- moved R2 237.3 mm to (126.8, 63.4)
- moved R1 237.3 mm to (126.8, 61.9), turned to 180 degrees
- moved R7 233.1 mm to (132.8, 60.9), turned to 180 degrees
- moved R6 232.4 mm to (132.8, 63.9)
- moved R5 232.2 mm to (132.8, 62.4), turned to 180 degrees
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Connections:
- D2 pad 3: /RP2350_Main/USB- -> /RP2350_Main/USB+
- D2 pad 4: /RP2350_Main/USB+ -> /RP2350_Main/USB-
Other:
- board outline added: 100 x 80 mm
