File: LogicAnalyzer_RP2350/LogicAnalyzer_RP2350/RP2350_Main.kicad_sch (KiCad schematic)
At the start: 62 parts, among them J2 SM03B-SRSS-TB, SW1 SW_MEC_5G, SW2 SW_MEC_5G, U3 W25Q128JVS, U4 RP2350A, Y1 12Mhz

Commit message: Routing for Micro Controller Section Done
Parts:
- C10, C11: footprint Capacitor_SMD:C_0402_1005Metric_Pad0.74x0.62mm_HandSolder -> Capacitor_0402 Small Pads for RP2350 VREG:C_0402_1005Metric_small_pads
- L3: footprint ABRACON AOTA-B201610S3R3-101-T:AOTAB201610S3R3101T -> Inductor_RP2350_Foot Print:L_pol_2016
Changed lines of the file:
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@@
 			)
 		)
-		(property "Footprint" "Capacitor_SMD:C_0402_1005Metric_Pad0.74x0.62mm_HandSolder"
+		(property "Footprint" "Capacitor_0402 Small Pads for RP2350 VREG:C_0402_1005Metric_small_pads"
 			(at 101.6 102.87 0)
 			(hide yes)
@@
 			)
 		)
-		(property "Footprint" "ABRACON AOTA-B201610S3R3-101-T:AOTAB201610S3R3101T"
+		(property "Footprint" "Inductor_RP2350_Foot Print:L_pol_2016"
 			(at 33.35 118.11 0)
 			(hide yes)
@@
 			)
 		)
-		(property "Footprint" "Capacitor_SMD:C_0402_1005Metric_Pad0.74x0.62mm_HandSolder"
+		(property "Footprint" "Capacitor_0402 Small Pads for RP2350 VREG:C_0402_1005Metric_small_pads"
 			(at 115.57 106.68 0)
 			(hide yes)

Commit message: Initial Routing Done, almost there
Parts:
- U4: footprint Package_DFN_QFN:QFN-60-1EP_7x7mm_P0.4mm_EP3.4x3.4mm_ThermalVias -> Package_DFN_QFN:QFN-60-1EP_7x7mm_P0.4mm_EP3.4x3.4mm
Changed lines of the file:
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@@
 			)
 		)
-		(property "Footprint" "Package_DFN_QFN:QFN-60-1EP_7x7mm_P0.4mm_EP3.4x3.4mm_ThermalVias"
+		(property "Footprint" "Package_DFN_QFN:QFN-60-1EP_7x7mm_P0.4mm_EP3.4x3.4mm"
 			(at 211.9787 150.368 0)
 			(hide yes)

Commit message: Almost there
Connections:
- net USB_BOOT renamed RP_BOOT
Changed lines of the file:
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@@
 		)
 	)
-	(label "USB_BOOT"
+	(label "RP_BOOT"
 		(at 64.77 109.22 90)
 		(effects

Commit message: DRcs and Warnings Cleared ready for release
Changed lines of the file:
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@@
+		)
+	)
+	(text_box "Skew between logic signals is 50 ps between the connector and the series resistor, and the maximum skew between the resistor and the RP2350 is 25 ps. This gives a total worst‑case skew of 75 ps across the 24 length‑matched channels.\nThis level of skew is suitable for synchronous digital signals up to ~1 GHz and logic rise times down to approximately 0.5-0.75 ns.Although this speed is beyond the actual analyser capabilities it is advised to use closest channels for synchronous digital signals\n"
+		(exclude_from_sim no)
+		(at 326.39 141.48 0)
+		(size 57.15 22.35)
+		(margins 0.9525 0.9525 0.9525 0.9525)
+		(stroke
+			(width 0)
+			(type solid)
+			(color 0 0 0 1)
+		)
+		(fill
+			(type color)
+			(color 72 72 72 1)
+		)
+		(effects
+			(font
+				(size 1.27 1.27)
+				(color 255 255 255 1)
+			)
+			(justify left top)
 		)
 	)
