File: LogicAnalyzer_RP2350/LogicAnalyzer_RP2350/_restore_backup_2026-08-09T20-16-18-365/FrontPanelInterface.kicad_sch (KiCad schematic)
At the start: 10 parts, among them J7 533984003, J8 2035571207, U11 ATtiny3216-S

Commit message: Clearing up some Import Errors
Connections:
- net GND: now also J7. (4), J8. (14); no longer J7.4 (MP), J7.5 (MP), J8.13 (MP), J8.14 (MP)
Changed lines of the file:
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@@
 		(pin "1"
 		)
-		(pin "5"
+		(pin ""
 		)
-		(pin "4"
+		(pin ""
 		)
 		(instances
@@
 		(pin "12"
 		)
-		(pin "14"
+		(pin ""
 		)
-		(pin "13"
+		(pin ""
 		)
 		(instances
