File: LogicAnalyzer_RP2350/LogicAnalyzer_RP2350/_restore_backup_2026-08-09T20-16-18-365/LogicAnalyzer_RP2350.kicad_pcb (KiCad board)
At the start: 4 copper layers, 143 parts, among them J1 2169890001, J2 SM03B-SRSS-TB, J3 SSW-106-02-TM-S-RA, J4 534269030, J5 534269030, J6 612050235221, J7 533984003, J8 2035571207, SW1 SW_MEC_5G, SW2 SW_MEC_5G, U1 NCP1117ST33T3G, U10 TXU0104PWR, U11 ATtiny3216-S, U2 TPS2552DRVR-1, U3 W25Q128JVS, U4 RP2350A, U5 TXU0104PWR, U6 TXU0104PWR, U7 TXU0104PWR, U8 TXU0104PWR, U9 TXU0104PWR, Y1 12Mhz

Commit message: Clearing up some Import Errors
Connections:
- J2 pad MP: GND -> (no net)
- J7 pad 4: GND -> (no net)
- J7 pad 5: GND -> (no net)
- J8 pad 13: GND -> (no net)
- J8 pad 14: GND -> (no net)
