File: LogicAnalyzer_RP2350/LogicAnalyzer_RP2350/_restore_backup_2026-08-09T20-16-18-365/RP2350_Main.kicad_sch (KiCad schematic)
At the start: 62 parts, among them J2 SM03B-SRSS-TB, SW1 SW_MEC_5G, SW2 SW_MEC_5G, U3 W25Q128JVS, U4 RP2350A, Y1 12Mhz

Commit message: Clearing up some Import Errors
Connections:
- net GND: now also J2. (MP); no longer J2.MP
Changed lines of the file:
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@@
 		(pin "1"
 		)
-		(pin "MP"
+		(pin ""
 		)
-		(pin "MP"
+		(pin ""
 		)
 		(instances
