File: LogicAnalyzer_RP2350/LogicAnalyzer_RP2350/_restore_backup_2026-08-09T20-16-18-365/USB & POWER.kicad_sch (KiCad schematic)
At the start: 21 parts, among them J1 2169890001, U1 NCP1117ST33T3G, U2 TPS2552DRVR-1

Commit message: Clearing up some Import Errors
Connections:
- net GND: no longer U2.GND_VIA (GND)
Changed lines of the file:
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@@
-	)
-	(junction
-		(at 220.98 64.77)
-		(diameter 0)
-		(color 0 0 0 0)
 	)
 	(junction
@@
 		(color 0 0 0 0)
 	)
-	(junction
-		(at 232.41 64.77)
-		(diameter 0)
-		(color 0 0 0 0)
-	)
 	(wire
 		(pts
@@
 	(wire
 		(pts
-			(xy 247.65 64.77) (xy 232.41 64.77)
+			(xy 247.65 64.77) (xy 228.6 64.77)
 		)
 		(stroke
@@
 	(wire
 		(pts
-			(xy 205.74 64.77) (xy 220.98 64.77)
+			(xy 205.74 64.77) (xy 224.79 64.77)
 		)
 		(stroke
@@
 	(wire
 		(pts
-			(xy 220.98 60.96) (xy 220.98 64.77)
-		)
-		(stroke
-			(width 0)
-			(type default)
-		)
-	)
-	(wire
-		(pts
 			(xy 118.11 102.87) (xy 114.3 102.87)
 		)
@@
 	(wire
 		(pts
-			(xy 232.41 60.96) (xy 232.41 64.77)
-		)
-		(stroke
-			(width 0)
-			(type default)
-		)
-	)
-	(wire
-		(pts
 			(xy 110.49 50.8) (xy 110.49 55.88)
 		)
@@
 	(wire
 		(pts
-			(xy 220.98 64.77) (xy 224.79 64.77)
-		)
-		(stroke
-			(width 0)
-			(type default)
-		)
-	)
-	(wire
-		(pts
 			(xy 58.42 143.51) (xy 81.28 143.51)
 		)
@@
 		(pts
 			(xy 54.61 49.53) (xy 83.82 49.53)
-		)
-		(stroke
-			(width 0)
-			(type default)
-		)
-	)
-	(wire
-		(pts
-			(xy 232.41 64.77) (xy 228.6 64.77)
 		)
 		(stroke
@@
 		(pin "3"
 		)
-		(pin "GND_VIA"
-		)
-		(pin "GND_VIA"
-		)
 		(instances
