File: LogicAnalyzer_RP2350/LogicAnalyzer_RP2350/_restore_backup_2026-08-12T19-34-57-893/LogicAnalyzer_RP2350.kicad_pcb (KiCad board)
At the start: 4 copper layers, 100 x 80 mm, 152 parts, among them J1 USB_C_Receptacle_USB2.0_16P, J2 SM03B-SRSS-TB, J3 SSW-106-02-TM-S-RA, J4 534269030, J5 534269030, J6 612050235221, J7 533984003, J8 2035571207, SW1 SW_MEC_5G, SW2 SW_MEC_5G, U1 NCP1117ST33T3G, U10 TXU0104PWR, U11 ATtiny3216-S, U2 TPS2552DRVR-1, U3 W25Q128JVS, U4 RP2350A, U5 TXU0104PWR, U6 TXU0104PWR, U7 TXU0104PWR, U8 TXU0104PWR, U9 TXU0104PWR, Y1 12Mhz

Commit message: TVS Swapped to more routing friendly, adjusting the Positions of TVs and Connectors
Parts:
- removed D14, D15, D16, D17, D18, D19, D20, D21, D22: SOT563_82400152, Diode_SMD_Wurth:D_Wurth_WE-TVS-SOT563
- D13, D4, D5: value SOT563_82400152 -> DFN3810-9L_824014885; footprint Diode_SMD_Wurth:D_Wurth_WE-TVS-SOT563 -> Diode_SMD_Wurth:D_Wurth_WE-TVS-DFN3810-9L
- moved FID3 272.3 mm to (374.1, 103.7)
- moved FID1 271.0 mm to (370.5, 103.7)
- moved FID2 226.3 mm to (370.5, 107.3)
- moved FID4 226.3 mm to (374.1, 107.3)
- moved FID6 226.3 mm to (377.6, 107.3)
- moved FID5 192.6 mm to (377.6, 103.7)
- moved D4 68.8 mm to (178.2, 116.9)
- moved D5 40.6 mm to (155.0, 116.9)
- moved U9 31.4 mm to (183.8, 109.4)
- moved C37 31.4 mm to (187.6, 105.1)
- moved C40 31.4 mm to (187.6, 111.9)
- moved C43 31.4 mm to (180.1, 111.9)
- moved C35 29.3 mm to (165.1, 111.6)
- moved C29 29.3 mm to (165.1, 105.1)
- moved U7 29.0 mm to (161.1, 109.4)
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Connections:
- D13 pad 1: /LevelShifters/DIN6 -> /LevelShifters/DIN7
- D13 pad 2: GND -> /LevelShifters/DIN5
- D13 pad 3: /LevelShifters/DIN5 -> GND
- D13 pad 4: /LevelShifters/DI5 -> /LevelShifters/DIN3
- D13 pad 5: +5V -> /LevelShifters/DIN1
- D13 pad 6: /LevelShifters/DI6 -> /LevelShifters/DIN2
- D4 pad 1: /LevelShifters/DIN2 -> /LevelShifters/DIN23
- D4 pad 2: GND -> /LevelShifters/DIN21
- D4 pad 3: /LevelShifters/DIN1 -> GND
- D4 pad 4: /LevelShifters/DI1 -> /LevelShifters/DIN19
- D4 pad 5: +5V -> /LevelShifters/DIN17
- D4 pad 6: /LevelShifters/DI2 -> /LevelShifters/DIN18
- D5 pad 1: /LevelShifters/DIN4 -> /LevelShifters/DIN15
- D5 pad 2: GND -> /LevelShifters/DIN13
- D5 pad 3: /LevelShifters/DIN3 -> GND
- D5 pad 4: /LevelShifters/DI3 -> /LevelShifters/DIN11
- D5 pad 5: +5V -> /LevelShifters/DIN9
- D5 pad 6: /LevelShifters/DI4 -> /LevelShifters/DIN10
- J6 pad 1: /LevelShifters/DI24 -> /LevelShifters/DIN1
- J6 pad 11: /LevelShifters/DI19 -> /LevelShifters/DIN6
- J6 pad 13: /LevelShifters/DI18 -> /LevelShifters/DIN7
- J6 pad 15: /LevelShifters/DI17 -> /LevelShifters/DIN8
- J6 pad 17: /LevelShifters/DI16 -> /LevelShifters/DIN9
- J6 pad 19: /LevelShifters/DI15 -> /LevelShifters/DIN10
- J6 pad 21: /LevelShifters/DI14 -> /LevelShifters/DIN11
- J6 pad 23: /LevelShifters/DI13 -> /LevelShifters/DIN12
- J6 pad 25: /LevelShifters/DI12 -> /LevelShifters/DIN13
- J6 pad 27: /LevelShifters/DI11 -> /LevelShifters/DIN14
- J6 pad 29: /LevelShifters/DI10 -> /LevelShifters/DIN15
- J6 pad 3: /LevelShifters/DI23 -> /LevelShifters/DIN2
- J6 pad 31: /LevelShifters/DI9 -> /LevelShifters/DIN16
- J6 pad 33: /LevelShifters/DI8 -> /LevelShifters/DIN17
- J6 pad 35: /LevelShifters/DI7 -> /LevelShifters/DIN18
- J6 pad 37: /LevelShifters/DI6 -> /LevelShifters/DIN19
- J6 pad 39: /LevelShifters/DI5 -> /LevelShifters/DIN20
- J6 pad 41: /LevelShifters/DI4 -> /LevelShifters/DIN21
- J6 pad 43: /LevelShifters/DI3 -> /LevelShifters/DIN22
- J6 pad 45: /LevelShifters/DI2 -> /LevelShifters/DIN23
- J6 pad 47: /LevelShifters/DI1 -> /LevelShifters/DIN24
- J6 pad 5: /LevelShifters/DI22 -> /LevelShifters/DIN3
- J6 pad 7: /LevelShifters/DI21 -> /LevelShifters/DIN4
- J6 pad 9: /LevelShifters/DI20 -> /LevelShifters/DIN5
- U10 pad 10: /LevelShifters/DIN21 -> /LevelShifters/DIN24
- U10 pad 11: /LevelShifters/DIN22 -> /LevelShifters/DIN23
- U10 pad 12: /LevelShifters/DIN23 -> /LevelShifters/DIN22
- U10 pad 13: /LevelShifters/DIN24 -> /LevelShifters/DIN21
- U10 pad 2: /LevelShifters/D24 -> /LevelShifters/D21
- U10 pad 3: /LevelShifters/D23 -> /LevelShifters/D22
- U10 pad 4: /LevelShifters/D22 -> /LevelShifters/D23
- U10 pad 5: /LevelShifters/D21 -> /LevelShifters/D24
- U5 pad 10: /LevelShifters/DIN1 -> /LevelShifters/DIN4
- U5 pad 11: /LevelShifters/DIN2 -> /LevelShifters/DIN3
- U5 pad 12: /LevelShifters/DIN3 -> /LevelShifters/DIN2
- U5 pad 13: /LevelShifters/DIN4 -> /LevelShifters/DIN1
- U5 pad 2: /LevelShifters/D4 -> /LevelShifters/D1
- U5 pad 3: /LevelShifters/D3 -> /LevelShifters/D2
- U5 pad 4: /LevelShifters/D2 -> /LevelShifters/D3
- U5 pad 5: /LevelShifters/D1 -> /LevelShifters/D4
- U6 pad 10: /LevelShifters/DIN5 -> /LevelShifters/DIN8
- U6 pad 11: /LevelShifters/DIN6 -> /LevelShifters/DIN7
- U6 pad 12: /LevelShifters/DIN7 -> /LevelShifters/DIN6
- U6 pad 13: /LevelShifters/DIN8 -> /LevelShifters/DIN5
- U6 pad 2: /LevelShifters/D8 -> /LevelShifters/D5
- U6 pad 3: /LevelShifters/D7 -> /LevelShifters/D6
- U6 pad 4: /LevelShifters/D6 -> /LevelShifters/D7
- U6 pad 5: /LevelShifters/D5 -> /LevelShifters/D8
- U7 pad 10: /LevelShifters/DIN9 -> /LevelShifters/DIN12
- U7 pad 11: /LevelShifters/DIN10 -> /LevelShifters/DIN11
- U7 pad 12: /LevelShifters/DIN11 -> /LevelShifters/DIN10
- U7 pad 13: /LevelShifters/DIN12 -> /LevelShifters/DIN9
- U7 pad 2: /LevelShifters/D12 -> /LevelShifters/D9
- U7 pad 3: /LevelShifters/D11 -> /LevelShifters/D10
- U7 pad 4: /LevelShifters/D10 -> /LevelShifters/D11
- U7 pad 5: /LevelShifters/D9 -> /LevelShifters/D12
- U8 pad 10: /LevelShifters/DIN13 -> /LevelShifters/DIN16
- U8 pad 11: /LevelShifters/DIN14 -> /LevelShifters/DIN15
- U8 pad 12: /LevelShifters/DIN15 -> /LevelShifters/DIN14
- U8 pad 13: /LevelShifters/DIN16 -> /LevelShifters/DIN13
- U8 pad 2: /LevelShifters/D16 -> /LevelShifters/D13
- U8 pad 3: /LevelShifters/D15 -> /LevelShifters/D14
- U8 pad 4: /LevelShifters/D14 -> /LevelShifters/D15
- U8 pad 5: /LevelShifters/D13 -> /LevelShifters/D16
- U9 pad 10: /LevelShifters/DIN17 -> /LevelShifters/DIN20
- U9 pad 11: /LevelShifters/DIN18 -> /LevelShifters/DIN19
- U9 pad 12: /LevelShifters/DIN19 -> /LevelShifters/DIN18
- U9 pad 13: /LevelShifters/DIN20 -> /LevelShifters/DIN17
- U9 pad 2: /LevelShifters/D20 -> /LevelShifters/D17
- U9 pad 3: /LevelShifters/D19 -> /LevelShifters/D18
- U9 pad 4: /LevelShifters/D18 -> /LevelShifters/D19
- U9 pad 5: /LevelShifters/D17 -> /LevelShifters/D20
Routing:
- net /RP2350_Main/XOUT: track 7.14 -> 0.00 mm
- net /RP2350_Main/XIN: track 6.10 -> 0.00 mm
- net /LevelShifters/DIN1: track 5.10 -> 0.00 mm
- net /LevelShifters/DIN4: track 5.06 -> 0.00 mm
- net /LevelShifters/DIN2: track 4.95 -> 0.00 mm
- net /LevelShifters/DIN3: track 4.93 -> 0.00 mm
- net Net-(U2-ILIM): track 3.72 -> 0.00 mm
- net /LevelShifters/DI7: track 3.08 -> 0.00 mm
- net /LevelShifters/DI6: track 3.08 -> 0.00 mm
- net /LevelShifters/DI4: track 3.08 -> 0.00 mm
- net /LevelShifters/DI2: track 3.08 -> 0.00 mm
- net /LevelShifters/DI14: track 3.08 -> 0.00 mm
- net /LevelShifters/DI12: track 3.08 -> 0.00 mm
- net /LevelShifters/DI11: track 3.08 -> 0.00 mm
- net /LevelShifters/DI10: track 3.08 -> 0.00 mm
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