File: LogicAnalyzer_RP2350/LogicAnalyzer_RP2350/_restore_backup_2026-08-12T19-34-57-893/RP2350_Main.kicad_sch (KiCad schematic)
At the start: 62 parts, among them J2 SM03B-SRSS-TB, SW1 SW_MEC_5G, SW2 SW_MEC_5G, U3 W25Q128JVS, U4 RP2350A, Y1 12Mhz

Commit message: TVS Swapped to more routing friendly, adjusting the Positions of TVs and Connectors
Parts:
- C10, C11, C12, C13, C14, C15, C16, C17, C18, C19, C20, C21, C22, C23, C24, C25, C26, C8, C9: footprint Capacitor_SMD:C_0402_1005Metric_Pad0.74x0.62mm_HandSolder -> Capacitor_SMD:C_0603_1608Metric_Pad1.08x0.95mm_HandSolder
- R14, R15, R16, R17, R19, R20, R21, R22, R23, R24, R25, R26, R27, R28, R29, R30, R31, R32, R33, R34, R35, R36, R37, R38, R39, R40, R41, R42: footprint Resistor_SMD:R_0402_1005Metric_Pad0.72x0.64mm_HandSolder -> Resistor_SMD:R_0603_1608Metric_Pad0.98x0.95mm_HandSolder
