File: LogicAnalyzer_RP2350/LogicAnalyzer_RP2350/_restore_backup_2026-08-12T19-34-57-893/USB & POWER.kicad_sch (KiCad schematic)
At the start: 21 parts, among them J1 USB_C_Receptacle_USB2.0_16P, U1 NCP1117ST33T3G, U2 TPS2552DRVR-1

Commit message: TVS Swapped to more routing friendly, adjusting the Positions of TVs and Connectors
Parts:
- removed J1: USB_C_Receptacle_USB2.0_16P, Connector_USB:USB_C_Receptacle_GCT_USB4105-xx-A_16P_TopMnt_Horizontal, symbol Connector:USB_C_Receptacle_USB2.0_16P
- added J1: 2169890001, USBC_Molex_2169890001:216989-0001_MOL, symbol USBC_Molex_2169890001:2169890001
Connections:
- net GND: now also J1.A1 (GND), J1.A12 (GND), J1.B1 (GND), J1.B12 (GND)
- net USB+: now also D2.4 (I/O2); no longer D2.3 (I/O1)
- net USB-: now also D2.3 (I/O1); no longer D2.4 (I/O2)
- net USBC+: now also J1.A6 (DP1), J1.B6 (DP2)
- net USBC-: now also J1.A7 (DN1), J1.B7 (DN2)
- net USBCC1: now also J1.A5 (CC1)
- net USBCC2: now also J1.B5 (CC2)
- net VBUS: now also J1.A4 (VBUS), J1.A9 (VBUS), J1.B4 (VBUS), J1.B9 (VBUS)
- no-connect marks 2 -> 0
Other:
- moved on the sheet: R1, R2
