File: LogicAnalyzer_RP2350/FrontPanel/FrontPanelPCB/FrontPanelPCB.kicad_pcb (KiCad board)
At the start: 2 copper layers, 95 x 42.6 mm, 29 parts, among them J1 2035571207, SW1 MTL-21-10

Commit message: DRCs Done
Parts:
- added REF**: OSHW-Logo_5.7x6mm_SilkScreen, Symbol:OSHW-Logo_5.7x6mm_SilkScreen, F.Cu at (157.8, 114.6)
- added REF**: ESD-Logo_6.6x6mm_SilkScreen, Symbol:ESD-Logo_6.6x6mm_SilkScreen, F.Cu at (107.3, 108.2)
- added REF**: KiCad-Logo2_5mm_SilkScreen, Symbol:KiCad-Logo2_5mm_SilkScreen, F.Cu at (110.9, 84.0)
- moved TP1 0.10 mm to (98.5, 107.0)
Connections:
- SW1 pad 1: +5V -> /VREF
- SW1 pad 2: +3.3V -> +5V
- SW1 pad 3: /EXTVREF -> +3.3V
- SW1 pad 4: unconnected-(SW1-Pad4) -> /EXTVREF
- SW1 pad 8: /VREF -> unconnected-(SW1-Pad8)
Routing:
- net /EXTVREF: track 0.00 -> 85.0 mm, vias 0 -> 1
- net +3.3V: track 0.00 -> 84.4 mm, vias 0 -> 1
- net /LEDA: track 2.47 -> 80.5 mm, vias 0 -> 3
- net /VREF: track 0.00 -> 75.3 mm, vias 0 -> 1
- net +5V: track 30.0 -> 78.3 mm, vias 8 -> 10
- net /SDA: track 0.00 -> 38.7 mm
- net /SCL: track 0.00 -> 34.1 mm
- net /LEDB: track 0.00 -> 16.0 mm, vias 0 -> 1
- net /LEDC: track 0.00 -> 14.8 mm, vias 0 -> 1
- net Net-(D7-DOUT): track 9.26 -> 11.3 mm
- net GND: vias 16 -> 252
- added copper zone on B.Cu, net GND
- added copper zone on F.Cu, net GND
Other:
- rule pad_to_mask_clearance: 0 -> 0.035
