File: LogicAnalyzer_RP2350/FrontPanel/FrontPanelPCB/FrontPanelPCB.kicad_sch (KiCad schematic)
At the start: 29 parts, among them J1 2035571207, SW1 MTL-21-10

Commit message: DRCs Done
Parts:
- removed H5, H7: M2.5, MountingHole:MountingHole_2.7mm_M2.5_Pad_Via, symbol Mechanical:MountingHole_Pad_MP
- added H1, H3: M2.5, MountingHole:MountingHole_2.7mm_M2.5_Pad_TopBottom, symbol Mechanical:MountingHole_Pad_MP
- H2: renamed from H6; footprint MountingHole:MountingHole_2.7mm_M2.5_Pad_Via -> MountingHole:MountingHole_2.7mm_M2.5_Pad_TopBottom
- H4: footprint MountingHole:MountingHole_2.7mm_M2.5_Pad_Via -> MountingHole:MountingHole_2.7mm_M2.5_Pad_TopBottom
Connections:
- net +3.3V: now also SW1.3; no longer SW1.2
- net +5V: now also SW1.2; no longer SW1.1
- net EXTVREF: now also SW1.4; no longer SW1.3
- net GND: now also H1.1, H3.1
- net VREF: now also SW1.1; no longer SW1.8
